Commit message: Use self.get_clock
Signed-off-by: Hunter L. Allen <hunter.allen@ghostrobotics.io>

File: create_description/urdf/create.urdf.xacro (robot description, xacro)
@@ -255,8 +255,8 @@
 	  </link>
 	  <!-- Simulation sensors -->
-	  <sim_create/>
-	  <sim_create_wall_sensor/>
-	  <sim_create_cliff_sensors/>
-    <sim_imu/>
+	  <xacro:sim_create/>
+	  <xacro:sim_create_wall_sensor/>
+	  <xacro:sim_create_cliff_sensors/>
+	  <xacro:sim_imu/>
   </xacro:macro>
 </robot>

File: create_description/urdf/create_gazebo.urdf.xacro (robot description, xacro)
@@ -1,20 +1,20 @@
 <?xml version="1.0"?>
 <robot xmlns:xacro="http://ros.org/wiki/xacro" name="turtlebot_gazebo">
-	<xacro:macro name="sim_create">
-	  <gazebo>
-	    <plugin name="create_controller" filename="libgazebo_ros_create.so">
-	      <alwaysOn>true</alwaysOn>
-	      <node_namespace>turtlebot_node</node_namespace>
-	      <left_wheel_joint>left_wheel_joint</left_wheel_joint>
-	      <right_wheel_joint>right_wheel_joint</right_wheel_joint>
-	      <front_castor_joint>front_castor_joint</front_castor_joint>
-	      <rear_castor_joint>rear_castor_joint</rear_castor_joint>
-	      <wheel_separation>.260</wheel_separation>
-	      <wheel_diameter>0.066</wheel_diameter>
-	      <base_geom>base_footprint_collision_base_link</base_geom>
-	      <updateRate>40</updateRate>
-	      <torque>1.0</torque>
-	    </plugin>
-	  </gazebo>
+  <xacro:macro name="sim_create">
+    <gazebo>
+      <plugin name="create_controller" filename="libgazebo_ros_create.so">
+	<alwaysOn>true</alwaysOn>
+	<node_namespace>turtlebot_node</node_namespace>
+	<left_wheel_joint>left_wheel_joint</left_wheel_joint>
+	<right_wheel_joint>right_wheel_joint</right_wheel_joint>
+	<front_castor_joint>front_castor_joint</front_castor_joint>
+	<rear_castor_joint>rear_castor_joint</rear_castor_joint>
+	<wheel_separation>.260</wheel_separation>
+	<wheel_diameter>0.066</wheel_diameter>
+	<base_geom>base_footprint_collision_base_link</base_geom>
+	<updateRate>40</updateRate>
+	<torque>1.0</torque>
+      </plugin>
+    </gazebo>
     <gazebo reference="left_wheel_link">
       <mu1>1.0</mu1>
@@ -49,21 +49,21 @@
       <maxVel>1.0</maxVel>
     </gazebo>
-	</xacro:macro>
-	<xacro:macro name="sim_imu">
-	  <gazebo>
-	    <plugin name="imu_controller" filename="libgazebo_ros_imu.so">
-	      <alwaysOn>true</alwaysOn>
-	      <updateRate>30</updateRate>
-	      <bodyName>gyro_link</bodyName>
-	      <topicName>imu/data</topicName>
+  </xacro:macro>
+  <xacro:macro name="sim_imu">
+    <gazebo>
+      <plugin name="imu_controller" filename="libgazebo_ros_imu.so">
+	<alwaysOn>true</alwaysOn>
+	<updateRate>30</updateRate>
+	<bodyName>gyro_link</bodyName>
+	<topicName>imu/data</topicName>
         <serviceName>imu/is_calibrated</serviceName>
-	      <gaussianNoise>${0.0017*0.0017}</gaussianNoise>
+	<gaussianNoise>${0.0017*0.0017}</gaussianNoise>
         <xyzOffsets>0 0 0</xyzOffsets>
         <rpyOffsets>0 0 0</rpyOffsets>
       </plugin>
-	  </gazebo>
-	</xacro:macro>
-	<xacro:macro name="sim_create_wall_sensor">
-	  <gazebo reference="wall_sensor_link">
+    </gazebo>
+  </xacro:macro>
+  <xacro:macro name="sim_create_wall_sensor">
+    <gazebo reference="wall_sensor_link">
       <sensor type="ray" name="wall_sensor">
         <always_on>true</always_on>
@@ -87,8 +87,8 @@
         </ray>
       </sensor>
-	  </gazebo>
-	</xacro:macro>
-	<xacro:macro name="sim_create_cliff_sensors">
-	  <gazebo reference="left_cliff_sensor_link">
+    </gazebo>
+  </xacro:macro>
+  <xacro:macro name="sim_create_cliff_sensors">
+    <gazebo reference="left_cliff_sensor_link">
       <sensor type="ray" name="left_cliff_sensor">
         <always_on>true</always_on>
@@ -112,6 +112,6 @@
         </ray>
       </sensor>
-	  </gazebo>
-	  <gazebo reference="right_cliff_sensor_link">
+    </gazebo>
+    <gazebo reference="right_cliff_sensor_link">
       <sensor type="ray" name="right_cliff_sensor">
         <always_on>true</always_on>
@@ -135,6 +135,6 @@
         </ray>
       </sensor>
-	  </gazebo>
-	  <gazebo reference="leftfront_cliff_sensor_link">
+    </gazebo>
+    <gazebo reference="leftfront_cliff_sensor_link">
       <sensor type="ray" name="leftfront_cliff_sensor">
         <always_on>true</always_on>
@@ -158,6 +158,6 @@
         </ray>
       </sensor>
-	  </gazebo>
-	  <gazebo reference="rightfront_cliff_sensor_link">
+    </gazebo>
+    <gazebo reference="rightfront_cliff_sensor_link">
       <sensor type="ray" name="rightfront_cliff_sensor">
         <always_on>true</always_on>
@@ -181,5 +181,5 @@
         </ray>
       </sensor>
-	  </gazebo>
-	</xacro:macro>
+    </gazebo>
+  </xacro:macro>
 </robot>
