Commit message: First running version with RPLIDAR on ROS2 galactic

File: create_description/urdf/create_nolaser.urdf.xacro (robot description, xacro)
@@ -235,24 +235,4 @@
 	    </inertial>
 	  </link>
-	  <joint name="laser_joint" type="fixed">
-	    <origin xyz="-0.065 0 0.075" rpy="0 0 0" />
-	    <parent link="base_link" />
-	    <child link="laser" />
-	  </joint>
-	  <link name="laser">
-	    <visual>
-	      <geometry>
-	        <box size="0.02 0.035 0.002" />
-	      </geometry>
-	      <material name="Green" />
-	    </visual>
-	    <inertial>
-	      <mass value="0.001" />
-	      <origin xyz="0 0 0" />
-	      <inertia ixx="0.0001" ixy="0.0" ixz="0.0"
-	        iyy="0.0001" iyz="0.0"
-	        izz="0.0001" />
-	    </inertial>
-	  </link>
 	  <!-- Simulation sensors -->
 	  <!--
